Commit message: bike position and kickstand

File: assets/bicycle_top_tube/bike_top_tube_vscode.urdf (robot description, URDF)
Before this commit: robot bike_top_tube_vscode, 4 links, 3 joints
Links:
- added link rear_support_left, mass 0.3; collision box size=0.02 0.4 0.02; visual box size=0.02 0.4 0.02
- added link rear_support_right, mass 0.3; collision box size=0.02 0.4 0.02; visual box size=0.02 0.4 0.02
- link back_wheel_1: mass None -> 1.0; geometry collision mesh filename=meshes/back_wheel_1.STL scale=0.001 0.001 0.001; visual mesh filename=meshes/back_wheel_1.STL scale=0.001 0.001 0.001
- link frame: mass None -> 2.0; geometry collision mesh filename=meshes/frame.STL scale=0.001 0.001 0.001; visual mesh filename=meshes/frame.STL scale=0.001 0.001 0.001
- link front_fork_1: mass None -> 1.0; geometry collision mesh filename=meshes/front_fork_1.STL scale=0.001 0.001 0.001; visual mesh filename=meshes/front_fork_1.STL scale=0.001 0.001 0.001
- link front_wheel_1: mass None -> 1.0; geometry collision mesh filename=meshes/front_wheel_1.STL scale=0.001 0.001 0.001; visual mesh filename=meshes/front_wheel_1.STL scale=0.001 0.001 0.001
Joints:
- added joint RearSupportLeft: type fixed, parent frame, child rear_support_left, origin xyz=-0.84811 0.08 -0.567533 rpy=0 0 0
- added joint RearSupportRight: type fixed, parent frame, child rear_support_right, origin xyz=-0.84811 -0.08 -0.567533 rpy=0 0 0
- joint Rev1: type continuous -> fixed
- joint Rev2: type continuous -> fixed
- joint Rev3: type continuous -> fixed

Commit message: Scale isomorphic settings

File: assets/bicycle_top_tube/bike_top_tube_vscode.urdf (robot description, URDF)
Before this commit: robot bike_top_tube, 6 links, 5 joints
Links:
- added link bike_root, mass 0.001; visual sphere radius=0.03
Joints:
- added joint BikeRootToFrame: type fixed, parent bike_root, child frame, origin xyz=0.33655284 0.000000 0.11421625 rpy=0 0 0
