Commit message: go back to original&run base only

File: assets/bicycle_top_tube/bike_top_tube_vscode.urdf (robot description, URDF)
Before this commit: robot bike_top_tube, 7 links, 6 joints
Links:
- link rear_support_left: geometry collision box size=0.12 1.2 0.02; visual box size=0.12 1.2 0.02
- link rear_support_right: geometry collision box size=0.12 1.2 0.02; visual box size=0.12 1.2 0.02
Joints:
- joint RearSupportLeft: origin xyz=-0.84811 0.08 -0.567533 rpy=0 0 0 -> xyz=0 0 0 rpy=0 0 0
- joint RearSupportRight: origin xyz=-0.84811 -0.08 -0.567533 rpy=0 0 0 -> xyz=0 0 0 rpy=0 0 0

File: assets/bicycle_top_tube/bikered.urdf (robot description, URDF)
Before this commit: robot bikered, 4 links, 3 joints
Links:
- link bike_root: geometry 
- link rear_support_left: geometry collision box size=0.12 1.2 0.02; visual box size=0.12 1.2 0.02
- link rear_support_right: geometry collision box size=0.12 1.2 0.02; visual box size=0.12 1.2 0.02
Joints:
- joint RearSupportLeft: origin xyz=-0.2 -1 -1.05 rpy=0 0 1.5 -> xyz=0 0 0 rpy=0 0 0
- joint RearSupportRight: origin xyz=0.2 -1 -1.05 rpy=0 0 1.5 -> xyz=0 0 0 rpy=0 0 0
