Commit message: urdf

File: assets/bicycle_top_tube/bikered.urdf (robot description, URDF)
Before this commit: robot bikered, 2 links, 1 joints
Links:
- added link rear_support_left, mass 0.3; collision box size=0.02 0.4 0.02; visual box size=0.02 0.4 0.02
- added link rear_support_right, mass 0.3; collision box size=0.02 0.4 0.02; visual box size=0.02 0.4 0.02
Joints:
- added joint RearSupportLeft: type fixed, parent bike_root, child rear_support_left, origin xyz=-0.2 -1 -1 rpy=0 0 1.5
- added joint RearSupportRight: type fixed, parent bike_root, child rear_support_right, origin xyz=0.2 -1 -1 rpy=0 0 1.5

Commit message: first training

File: assets/bicycle_top_tube/bikered.urdf (robot description, URDF)
Before this commit: robot bikered, 4 links, 3 joints
Joints:
- joint RearSupportLeft: origin xyz=-0.2 -1 -1 rpy=0 0 1.5 -> xyz=-0.2 -1 -1.05 rpy=0 0 1.5
- joint RearSupportRight: origin xyz=0.2 -1 -1 rpy=0 0 1.5 -> xyz=0.2 -1 -1.05 rpy=0 0 1.5
